File: PCB Designs/First Design/First Design.kicad_pcb (KiCad board)
At the start: 2 copper layers, 12 parts, among them J1 Conn_01x04, J2 Conn_01x04, U1 ATtiny13-20S

Commit message: Alot of uploads
Other:
- board text added: "Def no virus"
- board text added: "Very Safe USB"
