File: PCB Designs/Oscillator/Oscillator.kicad_sch (KiCad schematic)
At the start: 7 parts, among them Q3 2N2222A, Q4 2N2222A

Commit message: Changed Something (i have no idea what)
Parts:
- BT1: footprint (none) -> Battery:BatteryHolder_Bulgin_BX0034_1xAAA
- C2: value C -> 100u; footprint (none) -> Capacitor_SMD:CP_Elec_10x10
- D1, D2: footprint (none) -> LED_THT:LED_D3.0mm
- Q3, Q4: footprint 2N2222A:TO92254P470H750-3 -> Transisto:TO92254P470H750-3
- R1: footprint (none) -> Resistor_THT:R_Axial_DIN0204_L3.6mm_D1.6mm_P2.54mm_Vertical
Changed lines of the file:
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@@
 			)
 		)
-		(property "Footprint" ""
+		(property "Footprint" "LED_THT:LED_D3.0mm"
 			(at 118.11 91.44 0)
 			(hide yes)
@@
 			)
 		)
-		(property "Footprint" ""
+		(property "Footprint" "Battery:BatteryHolder_Bulgin_BX0034_1xAAA"
 			(at 166.37 108.966 90)
 			(hide yes)
@@
 			)
 		)
-		(property "Footprint" ""
+		(property "Footprint" "Resistor_THT:R_Axial_DIN0204_L3.6mm_D1.6mm_P2.54mm_Vertical"
 			(at 121.412 57.15 90)
 			(hide yes)
@@
 			)
 		)
-		(property "Footprint" ""
+		(property "Footprint" "LED_THT:LED_D3.0mm"
 			(at 140.97 91.44 0)
 			(hide yes)
@@
 			)
 		)
-		(property "Value" "C"
+		(property "Value" "100u"
 			(at 130.81 48.26 90)
 			(show_name no)
@@
 			)
 		)
-		(property "Footprint" ""
+		(property "Footprint" "Capacitor_SMD:CP_Elec_10x10"
 			(at 134.62 52.3748 0)
 			(hide yes)
@@
 			)
 		)
-		(property "Footprint" "2N2222A:TO92254P470H750-3"
+		(property "Footprint" "Transisto:TO92254P470H750-3"
 			(at 118.11 71.12 0)
 			(hide yes)
@@
 			)
 		)
-		(property "Footprint" "2N2222A:TO92254P470H750-3"
+		(property "Footprint" "Transisto:TO92254P470H750-3"
 			(at 140.97 71.12 0)
 			(hide yes)
