File: PCB Designs/Complex ESP 32/Main Practice/UI.kicad_sch (KiCad schematic)
At the start: 11 parts, among them J5 Conn_01x04_Pin, J6 Conn_01x05_Pin, Q2 BC817, Q3 BC817

Commit message: Started Schematics of footprint
Parts:
- S1, S2: footprint USLPT2819DT2TR:SW_USLPT2819DT2TR -> Footprints:SW_USLPT2819DT2TR
Changed lines of the file:
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@@
 			)
 		)
-		(property "Footprint" "USLPT2819DT2TR:SW_USLPT2819DT2TR"
+		(property "Footprint" "Footprints:SW_USLPT2819DT2TR"
 			(at 128.27 29.21 0)
 			(hide yes)
@@
 			)
 		)
-		(property "Footprint" "USLPT2819DT2TR:SW_USLPT2819DT2TR"
+		(property "Footprint" "Footprints:SW_USLPT2819DT2TR"
 			(at 88.9 29.21 0)
 			(hide yes)
